Commit message: Refina o pacote ROS 2: curva do motor, sensor de contato e odometria de referência
Três lacunas de fidelidade do primeiro corte do workspace.

Tração por esforço, com a curva real do motorredutor
Com interface de velocidade o ros2_control pedia rotação e o Gazebo entregava
qualquer torque até o limite da junta: o motor simulado tinha torque de stall a
1,53 m/s e o rover subiria escadas que o motorredutor real não sustenta — a
margem de 1,61 calculada no dimensionamento nunca era exercida. Agora a
interface é de esforço e o nó `tracao` converte velocidade desejada em torque
saturado pelo que o motor consegue entregar naquela rotação e tensão, com
queda de tensão do pack, modelo I²t por motor e PI com anti-windup (sem ele o
integrador carrega na escada e o rover dispara ao engatar).

Sensor de contato nas rodas
As pontas dos raios viraram colisões nomeadas e são referenciadas por um sensor
de contato por roda. É o que permite ver ONDE a roda toca — nariz, piso ou face
do espelho. O apoio na face do espelho é o modo de falha do achado A-01; sem
instrumentar o contato ele apareceria apenas como "o rover não subiu".

Odometria de verdade-terreno
Plugin de odometria no modelo, publicando a referência contra a qual medir o
erro da odometria por encoder — que a complacência do C-STS degrada em 30° de
atraso sob torque nominal. É o ensaio ENS-15, executável antes do hardware.

156 testes no total; 74 validam o pacote ROS sem ROS instalado, incluindo a
comparação ponto a ponto da curva do motor com simulador_python.powertrain.

Co-Authored-By: Claude Opus 5 <noreply@anthropic.com>
Claude-Session: https://claude.ai/code/session_011fV62gn6qdenHarLpSfQWB

File: ros2_ws/src/rover_frugal_description/urdf/rover_frugal.urdf.xacro (robot description, xacro)
@@ -34,4 +34,5 @@
   <xacro:property name="POS"  value="${cfg['posicoes_rodas']}"/>
   <xacro:property name="ESF"  value="${cfg['colisao_raios']}"/>
+  <xacro:property name="PONTAS" value="${cfg['colisao_pontas']}"/>
   <xacro:property name="malhas" value="package://rover_frugal_description/meshes"/>
   <xacro:property name="com_aro" value="$(arg aro_elastico)"/>
@@ -55,4 +56,17 @@
        O casco convexo da malha da roda é um disco: usar <mesh> como colisão
        apagaria a geometria de raios de que todo o projeto depende. -->
+  <!-- Pontas dos raios: colisões NOMEADAS, para o sensor de contato referenciar.
+       É a ponta que engata no nariz do degrau; saber onde ela toca (nariz, piso
+       ou face do espelho) é o que distingue "subiu" de "escorregou". -->
+  <xacro:macro name="esferas_pontas" params="prefixo lista sinal indice:=0">
+    <xacro:if value="${lista != []}">
+      <collision name="ponta_${prefixo}_${indice}">
+        <origin xyz="${lista[0][0]} 0 ${sinal * lista[0][1]}" rpy="0 0 0"/>
+        <geometry><sphere radius="${lista[0][2]}"/></geometry>
+      </collision>
+      <xacro:esferas_pontas prefixo="${prefixo}" lista="${lista[1:]}"
+                            sinal="${sinal}" indice="${indice + 1}"/>
+    </xacro:if>
+  </xacro:macro>
   <xacro:macro name="esferas_raios" params="lista sinal">
     <xacro:if value="${lista != []}">
@@ -214,5 +228,5 @@
         <!-- Com o aro montado a roda tem superfície contínua de rolamento:
              um cilindro no raio efetivo (r_max menos a deflexão estática). -->
-        <collision>
+        <collision name="aro_${prefixo}">
           <origin xyz="0 0 0" rpy="${pi/2} 0 0"/>
           <geometry>
@@ -223,4 +237,5 @@
       <xacro:unless value="${com_aro}">
         <xacro:esferas_raios lista="${ESF}" sinal="${lado}"/>
+        <xacro:esferas_pontas prefixo="${prefixo}" lista="${PONTAS}" sinal="${lado}"/>
       </xacro:unless>
     </link>
@@ -245,4 +260,22 @@
       <maxVel>0.5</maxVel>
       <material>Gazebo/Orange</material>
+      <!-- Sensor de contato: publica ONDE a roda toca. Sem ele, o apoio na face
+           do espelho (o modo de falha do achado A-01) apareceria apenas como
+           "o rover não subiu", sem dizer por quê. -->
+      <sensor name="contato_${prefixo}" type="contact">
+        <always_on>true</always_on>
+        <update_rate>100</update_rate>
+        <topic>contatos</topic>
+        <contact>
+          <xacro:if value="${com_aro}">
+            <collision>aro_${prefixo}</collision>
+          </xacro:if>
+          <xacro:unless value="${com_aro}">
+            <collision>ponta_${prefixo}_0</collision>
+            <collision>ponta_${prefixo}_1</collision>
+            <collision>ponta_${prefixo}_2</collision>
+          </xacro:unless>
+        </contact>
+      </sensor>
     </gazebo>
   </xacro:macro>
@@ -276,4 +309,16 @@
     <material>Gazebo/BlueTransparent</material>
   </gazebo>
+  <!-- Odometria de VERDADE-TERRENO. Não é a odometria do rover: é a referência
+       contra a qual medir o erro da odometria por encoder (ensaio ENS-15), que
+       a complacência do C-STS degrada. -->
+  <gazebo>
+    <plugin filename="gz-sim-odometry-publisher-system"
+            name="gz::sim::systems::OdometryPublisher">
+      <odom_frame>odom</odom_frame>
+      <robot_base_frame>base_footprint</robot_base_frame>
+      <odom_publish_frequency>50</odom_publish_frequency>
+      <dimensions>3</dimensions>
+    </plugin>
+  </gazebo>
   <xacro:include filename="$(find rover_frugal_description)/urdf/sensores.gazebo.xacro"/>
   <!-- ==================================================================== -->
@@ -295,8 +340,11 @@
           <state_interface name="effort"/>
         </joint>
+        <!-- Tração por ESFORÇO, não por velocidade: é o nó `tracao` que aplica
+             a curva torque-velocidade do motorredutor. Com interface de
+             velocidade o motor simulado teria torque de stall a 1,5 m/s. -->
         <joint name="tracao_${prefixo}">
-          <command_interface name="velocity">
-            <param name="min">${-J['tracao']['velocidade_maxima']}</param>
-            <param name="max">${J['tracao']['velocidade_maxima']}</param>
+          <command_interface name="effort">
+            <param name="min">${-J['tracao']['esforco_maximo']}</param>
+            <param name="max">${J['tracao']['esforco_maximo']}</param>
           </command_interface>
           <state_interface name="position"/>
